File: KiCAD Boards/LineFollower_V2/2_PSU.kicad_sch (KiCad schematic)
At the start: 36 parts, among them IC3 LMR36015FBRNXT, IC4 LMR36015FBRNXT, Q1 BC817, Q2 BC817, U1 HC-VH-2A-TW

Commit message: fix values, layout switchers
Parts:
- C10, C9: value 100nF -> 1uF
- C11, C14, C17, C19: value 100nF -> 220nF
- C12, C15, C18, C20, C23, C24, C25, C26: value 100nF -> 22uF; footprint Capacitor_SMD:C_0603_1608Metric -> Capacitor_SMD:C_0805_2012Metric
- C21, C22: value 100nF -> 20pF
- R10, R6, R7, R8: value 10K -> 100k
- R11: value 10K -> 24k9
- R9: value 10K -> 43k2
Connections:
- net +5V: now reaches C22.1, C24.1, C26.1, R10.2
- net +5V: now also L2.2
Other:
- moved on the sheet: L2
Changed lines of the file:
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@@
 	)
 	(junction
-		(at 200.66 101.6)
-		(diameter 0)
-		(color 0 0 0 0)
-	)
-	(junction
 		(at 139.7 105.41)
 		(diameter 0)
@@
 	)
 	(junction
+		(at 200.66 101.6)
+		(diameter 0)
+		(color 0 0 0 0)
+	)
+	(junction
 		(at 207.01 31.75)
 		(diameter 0)
@@
 	(wire
 		(pts
-			(xy 170.18 101.6) (xy 175.26 101.6)
+			(xy 170.18 101.6) (xy 174.0154 101.6)
 		)
 		(stroke
@@
 	(wire
 		(pts
+			(xy 214.63 100.33) (xy 214.63 101.6)
+		)
+		(stroke
+			(width 0)
+			(type default)
+		)
+	)
+	(wire
+		(pts
 			(xy 137.16 40.64) (xy 139.7 40.64)
 		)
@@
 	(wire
 		(pts
+			(xy 194.31 101.6) (xy 200.66 101.6)
+		)
+		(stroke
+			(width 0)
+			(type default)
+		)
+	)
+	(wire
+		(pts
 			(xy 124.46 105.41) (xy 123.19 105.41)
 		)
@@
 	(wire
 		(pts
-			(xy 214.63 101.6) (xy 214.63 99.06)
-		)
-		(stroke
-			(width 0)
-			(type default)
-		)
-	)
-	(wire
-		(pts
 			(xy 139.7 99.06) (xy 139.7 105.41)
 		)
@@
 	(wire
 		(pts
-			(xy 195.58 101.6) (xy 200.66 101.6)
-		)
-		(stroke
-			(width 0)
-			(type default)
-		)
-	)
-	(wire
-		(pts
 			(xy 128.27 50.8) (xy 128.27 63.5)
 		)
@@
 			)
 		)
-		(property "Value" "10K"
+		(property "Value" "100k"
 			(at 194.31 106.68 90)
 			(effects
@@
 			)
 		)
-		(property "Value" "10K"
+		(property "Value" "100k"
 			(at 109.22 52.07 0)
 			(effects
@@
 			)
 		)
-		(property "Value" "100nF"
+		(property "Value" "22uF"
 			(at 204.47 40.64 0)
 			(effects
@@
 			)
 		)
-		(property "Footprint" "Capacitor_SMD:C_0603_1608Metric"
+		(property "Footprint" "Capacitor_SMD:C_0805_2012Metric"
 			(at 207.01 39.37 0)
 			(effects
@@
 			)
 		)
-		(property "Value" "100nF"
+		(property "Value" "22uF"
 			(at 212.09 110.49 0)
 			(effects
@@
 			)
 		)
-		(property "Footprint" "Capacitor_SMD:C_0603_1608Metric"
+		(property "Footprint" "Capacitor_SMD:C_0805_2012Metric"
 			(at 214.63 109.22 0)
 			(effects
@@
 			)
 		)
-		(property "Value" "10K"
+		(property "Value" "43k2"
 			(at 200.66 57.15 90)
 			(effects
@@
 			)
 		)
-		(property "Value" "100nF"
+		(property "Value" "22uF"
 			(at 209.55 40.64 0)
 			(effects
@@
 			)
 		)
-		(property "Footprint" "Capacitor_SMD:C_0603_1608Metric"
+		(property "Footprint" "Capacitor_SMD:C_0805_2012Metric"
 			(at 212.09 39.37 0)
 			(effects
@@
 	)
 	(symbol
-		(lib_id "Robot druh-easyedapro:Power-5V")
-		(at 214.63 99.06 0)
-		(unit 1)
-		(exclude_from_sim no)
-		(in_bom yes)
-		(on_board yes)
-		(dnp no)
-		(property "Reference" "#PWR041"
-			(at 214.63 99.06 0)
-			(effects
-				(font
-					(size 1.27 1.27)
-				)
-				(hide yes)
-			)
-		)
-		(property "Value" "~"
-			(at 214.63 93.98 0)
-			(effects
-				(font
-					(size 1.27 1.27)
-				)
-			)
-		)
-		(property "Footprint" "Robot druh-easyedapro:"
-			(at 214.63 99.06 0)
-			(effects
-				(font
-					(size 1.27 1.27)
-				)
-				(hide yes)
-			)
-		)
-		(property "Datasheet" ""
-			(at 214.63 99.06 0)
-			(effects
-				(font
-					(size 1.27 1.27)
-				)
-				(hide yes)
-			)
-		)
-		(property "Description" "Power-5V"
-			(at 214.63 99.06 0)
-			(effects
-				(font
-					(size 1.27 1.27)
-				)
-				(hide yes)
-			)
-		)
-		(pin "1"
-		)
-		(instances
-			(project "LineFollower_V2"
-				(path "/76a20473-53d0-433c-9f05-17cd0a98178a/5d9dbd08-e291-4910-b472-c97ee13cd6ca"
-					(reference "#PWR041")
-					(unit 1)
-				)
-			)
-		)
-	)
-	(symbol
 		(lib_id "Robot druh-easyedapro:Ground-GND")
 		(at 121.92 110.49 270)
@@
 			)
 		)
-		(property "Value" "100nF"
+		(property "Value" "20pF"
 			(at 201.93 45.72 0)
 			(effects
@@
 			)
 		)
-		(property "Value" "10K"
+		(property "Value" "100k"
 			(at 198.12 46.99 0)
 			(effects
@@
 			)
 		)
-		(property "Value" "100nF"
+		(property "Value" "220nF"
 			(at 130.81 105.41 0)
 			(effects
@@
 			)
 		)
-		(property "Value" "100nF"
+		(property "Value" "22uF"
 			(at 130.81 110.49 0)
 			(effects
@@
 			)
 		)
-		(property "Footprint" "Capacitor_SMD:C_0603_1608Metric"
+		(property "Footprint" "Capacitor_SMD:C_0805_2012Metric"
 			(at 129.54 110.49 0)
 			(effects
@@
 			)
 		)
-		(property "Value" "100nF"
+		(property "Value" "220nF"
 			(at 179.07 38.1 0)
 			(effects
@@
 			)
 		)
-		(property "Value" "10K"
+		(property "Value" "24k9"
 			(at 203.2 127 90)
 			(effects
@@
 			)
 		)
-		(property "Value" "100nF"
+		(property "Value" "220nF"
 			(at 181.61 107.95 0)
 			(effects
@@
 			)
 		)
-		(property "Value" "100nF"
+		(property "Value" "1uF"
 			(at 121.92 60.96 0)
 			(effects
@@
 	)
 	(symbol
+		(lib_id "power:+5V")
+		(at 214.63 100.33 0)
+		(unit 1)
+		(exclude_from_sim no)
+		(in_bom yes)
+		(on_board yes)
+		(dnp no)
+		(fields_autoplaced yes)
+		(property "Reference" "#PWR041"
+			(at 214.63 104.14 0)
+			(effects
+				(font
+					(size 1.27 1.27)
+				)
+				(hide yes)
+			)
+		)
+		(property "Value" "+5V"
+			(at 214.63 95.25 0)
+			(effects
+				(font
+					(size 1.27 1.27)
+				)
+			)
+		)
+		(property "Footprint" ""
+			(at 214.63 100.33 0)
+			(effects
+				(font
+					(size 1.27 1.27)
+				)
+				(hide yes)
+			)
+		)
+		(property "Datasheet" ""
+			(at 214.63 100.33 0)
+			(effects
+				(font
+					(size 1.27 1.27)
+				)
+				(hide yes)
+			)
+		)
+		(property "Description" "Power symbol creates a global label with name \"+5V\""
+			(at 214.63 100.33 0)
+			(effects
+				(font
+					(size 1.27 1.27)
+				)
+				(hide yes)
+			)
+		)
+		(pin "1"
+		)
+		(instances
+			(project ""
+				(path "/76a20473-53d0-433c-9f05-17cd0a98178a/5d9dbd08-e291-4910-b472-c97ee13cd6ca"
+					(reference "#PWR041")
+					(unit 1)
+				)
+			)
+		)
+	)
+	(symbol
 		(lib_id "Robot druh-easyedapro:Ground-GND")
 		(at 187.96 43.18 90)
@@
 			)
 		)
-		(property "Value" "100nF"
+		(property "Value" "22uF"
 			(at 179.07 43.18 0)
 			(effects
@@
 			)
 		)
-		(property "Footprint" "Capacitor_SMD:C_0603_1608Metric"
+		(property "Footprint" "Capacitor_SMD:C_0805_2012Metric"
 			(at 177.8 43.18 0)
 			(effects
@@
 			)
 		)
-		(property "Value" "100nF"
+		(property "Value" "20pF"
 			(at 204.47 115.57 0)
 			(effects
@@
 			)
 		)
-		(property "Value" "100nF"
+		(property "Value" "22uF"
 			(at 181.61 113.03 0)
 			(effects
@@
 			)
 		)
-		(property "Footprint" "Capacitor_SMD:C_0603_1608Metric"
+		(property "Footprint" "Capacitor_SMD:C_0805_2012Metric"
 			(at 180.34 113.03 0)
 			(effects
@@
 	(symbol
 		(lib_id "Robot druh-easyedapro:XAL7030-103MEC_")
-		(at 175.26 101.6 0)
+		(at 174.0154 101.6 0)
 		(unit 1)
 		(exclude_from_sim no)
@@
 		(dnp no)
 		(property "Reference" "L2"
-			(at 184.15 104.14 0)
+			(at 182.9054 104.14 0)
 			(effects
 				(font
@@
 		)
 		(property "Value" "10uH"
-			(at 182.88 100.33 0)
+			(at 181.6354 100.33 0)
 			(effects
 				(font
@@
 		)
 		(property "Footprint" "easyEDA_footprints:XAL7030103MEC"
-			(at 175.26 101.6 0)
+			(at 174.0154 101.6 0)
 			(effects
 				(font
@@
 		)
 		(property "Datasheet" ""
-			(at 175.26 101.6 0)
+			(at 174.0154 101.6 0)
 			(effects
 				(font
@@
 		)
 		(property "Description" ""
-			(at 175.26 101.6 0)
+			(at 174.0154 101.6 0)
 			(effects
 				(font
@@
 			)
 		)
-		(property "Value" "100nF"
+		(property "Value" "220nF"
 			(at 128.27 35.56 0)
 			(effects
@@
 			)
 		)
-		(property "Value" "10K"
+		(property "Value" "100k"
 			(at 115.57 121.92 0)
 			(effects
@@
 			)
 		)
-		(property "Value" "100nF"
+		(property "Value" "1uF"
 			(at 124.46 130.81 0)
 			(effects
@@
 			)
 		)
-		(property "Value" "100nF"
+		(property "Value" "22uF"
 			(at 128.27 40.64 0)
 			(effects
@@
 			)
 		)
-		(property "Footprint" "Capacitor_SMD:C_0603_1608Metric"
+		(property "Footprint" "Capacitor_SMD:C_0805_2012Metric"
 			(at 127 40.64 0)
 			(effects
@@
 			)
 		)
-		(property "Value" "100nF"
+		(property "Value" "22uF"
 			(at 207.01 110.49 0)
 			(effects
@@
 			)
 		)
-		(property "Footprint" "Capacitor_SMD:C_0603_1608Metric"
+		(property "Footprint" "Capacitor_SMD:C_0805_2012Metric"
 			(at 209.55 109.22 0)
 			(effects

Commit message: some routing
Connections:
- net 3V3_SWITCHING_OUT: now also L1.2
- net GND: now also R11.1, R9.1
- net at C22.2, R10.1, R11.2: now also IC4.7 (FB)
- net at IC3.7 (FB): now also C21.2, R8.1, R9.2; no longer R9.1
Changed lines of the file:
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@@
 	)
 	(junction
-		(at 120.65 45.72)
+		(at 200.66 118.11)
 		(diameter 0)
 		(color 0 0 0 0)
 	)
 	(junction
-		(at 198.12 31.75)
+		(at 120.65 45.72)
 		(diameter 0)
 		(color 0 0 0 0)
@@
 	)
 	(junction
+		(at 198.12 31.75)
+		(diameter 0)
+		(color 0 0 0 0)
+	)
+	(junction
 		(at 214.63 116.84)
 		(diameter 0)
@@
 	)
 	(junction
+		(at 198.12 48.26)
+		(diameter 0)
+		(color 0 0 0 0)
+	)
+	(junction
 		(at 214.63 101.6)
 		(diameter 0)
@@
 	(wire
 		(pts
-			(xy 200.66 119.38) (xy 200.66 116.84)
+			(xy 200.66 119.38) (xy 200.66 118.11)
 		)
 		(stroke
@@
 	(wire
 		(pts
-			(xy 120.65 45.72) (xy 121.92 45.72)
+			(xy 198.12 48.26) (xy 198.12 46.99)
 		)
 		(stroke
@@
 	(wire
 		(pts
-			(xy 180.34 50.8) (xy 180.34 62.23)
+			(xy 120.65 45.72) (xy 121.92 45.72)
 		)
 		(stroke
@@
 	(wire
 		(pts
+			(xy 193.04 31.75) (xy 198.12 31.75)
+		)
+		(stroke
+			(width 0)
+			(type default)
+		)
+	)
+	(wire
+		(pts
+			(xy 200.66 118.11) (xy 200.66 116.84)
+		)
+		(stroke
+			(width 0)
+			(type default)
+		)
+	)
+	(wire
+		(pts
 			(xy 120.65 35.56) (xy 121.92 35.56)
 		)
@@
 	(wire
 		(pts
+			(xy 194.31 48.26) (xy 198.12 48.26)
+		)
+		(stroke
+			(width 0)
+			(type default)
+		)
+	)
+	(wire
+		(pts
 			(xy 121.92 50.8) (xy 121.92 48.26)
 		)
@@
 	(wire
 		(pts
+			(xy 195.58 120.65) (xy 195.58 118.11)
+		)
+		(stroke
+			(width 0)
+			(type default)
+		)
+	)
+	(wire
+		(pts
 			(xy 167.64 60.96) (xy 167.64 40.64)
 		)
@@
 	(wire
 		(pts
-			(xy 165.1 120.65) (xy 182.88 120.65)
+			(xy 165.1 120.65) (xy 195.58 120.65)
 		)
 		(stroke
@@
 	(wire
 		(pts
-			(xy 180.34 50.8) (xy 162.56 50.8)
+			(xy 162.56 50.8) (xy 194.31 50.8)
 		)
 		(stroke
@@
 	(wire
 		(pts
-			(xy 198.12 49.53) (xy 198.12 46.99)
+			(xy 198.12 49.53) (xy 198.12 48.26)
 		)
 		(stroke
@@
 	(wire
 		(pts
-			(xy 167.64 31.75) (xy 172.72 31.75)
+			(xy 167.64 31.75) (xy 172.7454 31.75)
 		)
 		(stroke
@@
 	(wire
 		(pts
-			(xy 193.04 31.75) (xy 198.12 31.75)
-		)
-		(stroke
-			(width 0)
-			(type default)
-		)
-	)
-	(wire
-		(pts
-			(xy 180.34 62.23) (xy 198.12 62.23)
-		)
-		(stroke
-			(width 0)
-			(type default)
-		)
-	)
-	(wire
-		(pts
 			(xy 134.62 105.41) (xy 139.7 105.41)
 		)
@@
 	(wire
 		(pts
-			(xy 167.64 38.1) (xy 162.56 38.1)
+			(xy 195.58 118.11) (xy 200.66 118.11)
 		)
 		(stroke
@@
 	(wire
 		(pts
-			(xy 187.96 113.03) (xy 187.96 107.95)
+			(xy 167.64 38.1) (xy 162.56 38.1)
 		)
 		(stroke
@@
 	(wire
 		(pts
-			(xy 134.62 110.49) (xy 139.7 110.49)
+			(xy 187.96 113.03) (xy 187.96 107.95)
 		)
 		(stroke
@@
 	(wire
 		(pts
-			(xy 137.16 29.21) (xy 137.16 35.56)
+			(xy 134.62 110.49) (xy 139.7 110.49)
 		)
 		(stroke
@@
 	(wire
 		(pts
-			(xy 139.7 99.06) (xy 139.7 105.41)
+			(xy 137.16 29.21) (xy 137.16 35.56)
 		)
 		(stroke
@@
 	(wire
 		(pts
-			(xy 182.88 120.65) (xy 182.88 132.08)
+			(xy 139.7 99.06) (xy 139.7 105.41)
 		)
 		(stroke
@@
 	(wire
 		(pts
-			(xy 182.88 132.08) (xy 200.66 132.08)
-		)
-		(stroke
-			(width 0)
-			(type default)
-		)
-	)
-	(wire
-		(pts
 			(xy 104.14 48.26) (xy 106.68 48.26)
 		)
@@
 	(wire
 		(pts
+			(xy 194.31 50.8) (xy 194.31 48.26)
+		)
+		(stroke
+			(width 0)
+			(type default)
+		)
+	)
+	(wire
+		(pts
 			(xy 198.12 46.99) (xy 198.12 44.45)
 		)
@@
 	(symbol
 		(lib_id "Robot druh-easyedapro:Ground-GND")
-		(at 190.5 113.03 90)
+		(at 190.5 113.03 0)
 		(unit 1)
 		(exclude_from_sim no)
@@
 		)
 		(property "Value" "GND"
-			(at 196.85 113.03 0)
+			(at 190.5 119.38 0)
 			(effects
 				(font
@@
 	(symbol
 		(lib_id "Robot druh-easyedapro:Ground-GND")
+		(at 200.66 132.08 0)
+		(unit 1)
+		(exclude_from_sim no)
+		(in_bom yes)
+		(on_board yes)
+		(dnp no)
+		(property "Reference" "#PWR0100"
+			(at 200.66 132.08 0)
+			(effects
+				(font
+					(size 1.27 1.27)
+				)
+				(hide yes)
+			)
+		)
+		(property "Value" "GND"
+			(at 200.66 138.43 0)
+			(effects
+				(font
+					(size 1.27 1.27)
+				)
+			)
+		)
+		(property "Footprint" "Robot druh-easyedapro:"
+			(at 200.66 132.08 0)
+			(effects
+				(font
+					(size 1.27 1.27)
+				)
+				(hide yes)
+			)
+		)
+		(property "Datasheet" ""
+			(at 200.66 132.08 0)
+			(effects
+				(font
+					(size 1.27 1.27)
+				)
+				(hide yes)
+			)
+		)
+		(property "Description" ""
+			(at 200.66 132.08 0)
+			(effects
+				(font
+					(size 1.27 1.27)
+				)
+				(hide yes)
+			)
+		)
+		(pin "1"
+		)
+		(instances
+			(project "LineFollower_V2"
+				(path "/76a20473-53d0-433c-9f05-17cd0a98178a/5d9dbd08-e291-4910-b472-c97ee13cd6ca"
+					(reference "#PWR0100")
+					(unit 1)
+				)
+			)
+		)
+	)
+	(symbol
+		(lib_id "Robot druh-easyedapro:Ground-GND")
+		(at 198.12 62.23 0)
+		(unit 1)
+		(exclude_from_sim no)
+		(in_bom yes)
+		(on_board yes)
+		(dnp no)
+		(property "Reference" "#PWR0101"
+			(at 198.12 62.23 0)
+			(effects
+				(font
+					(size 1.27 1.27)
+				)
+				(hide yes)
+			)
+		)
+		(property "Value" "GND"
+			(at 198.12 68.58 0)
+			(effects
+				(font
+					(size 1.27 1.27)
+				)
+			)
+		)
+		(property "Footprint" "Robot druh-easyedapro:"
+			(at 198.12 62.23 0)
+			(effects
+				(font
+					(size 1.27 1.27)
+				)
+				(hide yes)
+			)
+		)
+		(property "Datasheet" ""
+			(at 198.12 62.23 0)
+			(effects
+				(font
+					(size 1.27 1.27)
+				)
+				(hide yes)
+			)
+		)
+		(property "Description" ""
+			(at 198.12 62.23 0)
+			(effects
+				(font
+					(size 1.27 1.27)
+				)
+				(hide yes)
+			)
+		)
+		(pin "1"
+		)
+		(instances
+			(project "LineFollower_V2"
+				(path "/76a20473-53d0-433c-9f05-17cd0a98178a/5d9dbd08-e291-4910-b472-c97ee13cd6ca"
+					(reference "#PWR0101")
+					(unit 1)
+				)
+			)
+		)
+	)
+	(symbol
+		(lib_id "Robot druh-easyedapro:Ground-GND")
 		(at 214.63 119.38 0)
 		(unit 1)
@@
 	(symbol
 		(lib_id "Robot druh-easyedapro:Ground-GND")
-		(at 187.96 43.18 90)
+		(at 187.96 43.18 0)
 		(unit 1)
 		(exclude_from_sim no)
@@
 		)
 		(property "Value" "GND"
-			(at 194.31 43.18 0)
+			(at 187.96 49.53 0)
 			(effects
 				(font
@@
 	(symbol
 		(lib_id "Robot druh-easyedapro:IHLP2020BZER6R8M01_")
-		(at 172.72 31.75 0)
+		(at 172.7454 31.75 0)
 		(unit 1)
 		(exclude_from_sim no)
@@
 		(dnp no)
 		(property "Reference" "L1"
-			(at 181.61 34.29 0)
+			(at 181.6354 34.29 0)
 			(effects
 				(font
@@
 		)
 		(property "Value" "6.8uH"
-			(at 180.34 30.48 0)
+			(at 180.3654 30.48 0)
 			(effects
 				(font
@@
 		)
 		(property "Footprint" "easyEDA_footprints:INDPM5552X200N"
-			(at 172.72 31.75 0)
+			(at 172.7454 31.75 0)
 			(effects
 				(font
@@
 		)
 		(property "Datasheet" ""
-			(at 172.72 31.75 0)
+			(at 172.7454 31.75 0)
 			(effects
 				(font
@@
 		)
 		(property "Description" ""
-			(at 172.72 31.75 0)
+			(at 172.7454 31.75 0)
 			(effects
 				(font
