File: KiCAD Boards/LineFollower_V2/5_LGBT lighting.kicad_sch (KiCad schematic)
At the start: 10 parts

Commit message: fix values, layout switchers
Connections:
- net +5V: now reaches LED10.1 (VDD)
- net +5V: now also LED11.1 (VDD), LED12.1 (VDD), LED3.1 (VDD), LED4.1 (VDD), LED5.1 (VDD), LED6.1 (VDD), LED7.1 (VDD), LED8.1 (VDD), LED9.1 (VDD)
