File: KiCAD Boards/LineFollower_V2/6_Encoder interface.kicad_sch (KiCad schematic)
At the start: 10 parts, among them IC9 PCA9548APWR, U2 DIP_2*5PIN_80MIL

Commit message: fix values, layout switchers
Parts:
- R13, R14, R15, R16, R17, R18: value 10K -> 5k1
Changed lines of the file:
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@@
 			)
 		)
-		(property "Value" "10K"
+		(property "Value" "5k1"
 			(at 198.12 74.93 90)
 			(effects
@@
 			)
 		)
-		(property "Value" "10K"
+		(property "Value" "5k1"
 			(at 160.02 74.93 90)
 			(effects
@@
 			)
 		)
-		(property "Value" "10K"
+		(property "Value" "5k1"
 			(at 110.49 62.23 90)
 			(effects
@@
 			)
 		)
-		(property "Value" "10K"
+		(property "Value" "5k1"
 			(at 213.36 74.93 90)
 			(effects
@@
 			)
 		)
-		(property "Value" "10K"
+		(property "Value" "5k1"
 			(at 177.8 74.93 90)
 			(effects
@@
 			)
 		)
-		(property "Value" "10K"
+		(property "Value" "5k1"
 			(at 96.52 62.23 90)
 			(effects
