File: KiCAD Boards/LineFollower_V2/7_Sensor input.kicad_sch (KiCad schematic)
At the start: 5 parts, among them CON1 XDFC-0520-40P, IC5 74HC165BQ,115, IC6 74HC165BQ,115, IC7 74HC165BQ,115, IC8 74HC165BQ,115

Commit message: fix values, layout switchers
Connections:
- net 3V3: now reaches IC7.16 (VCC)
- net 3V3: now also IC5.16 (VCC), IC6.16 (VCC), IC8.16 (VCC)

Commit message: more routing
Parts:
- added C33, C34, C35, C36: 220nF, Capacitor_SMD:C_0603_1608Metric, symbol Robot druh-easyedapro:CAP
Connections:
- net VCC is gone; now on net 3V3: CON1.4, CON1.5
- net 3V3: now also C33.1, C34.1, C35.1, C36.1
- net DIR14: no longer IC7.5 (D6)
- net DIR15: now also IC7.5 (D6)
- net DIR17: no longer CON1.33, IC6.11 (D0)
- net DIR18: no longer CON1.34, IC6.12 (D1)
- net DIR19: no longer CON1.35, IC6.13 (D2)
- net DIR20: no longer CON1.36, IC6.14 (D3)
- net DIR21: no longer CON1.37, IC6.3 (D4)
- net DIR22: no longer CON1.38, IC6.4 (D5)
- net DIR23: no longer CON1.39, IC6.5 (D6)
- net DIR24: no longer CON1.40
- net GND: now also IC5.15 (CE#), IC5.17 (PAD), IC6.15 (CE#), IC6.17 (PAD), IC7.15 (CE#), IC7.17 (PAD), IC8.15 (CE#), IC8.17 (PAD), C33.2, C34.2, C35.2, C36.2
- net LOAD_Shift: now reaches IC7.1 (PL#)
- net LOAD_Shift: now also IC5.1 (PL#), IC6.1 (PL#), IC8.1 (PL#)
- net at IC7.10 (DS): now also IC8.9 (Q7)
- net CLK_Shift: now reaches IC7.2 (CP)
- net CLK_Shift: now also IC5.2 (CP), IC6.2 (CP), IC8.2 (CP)
- net at IC7.9 (Q7): now also IC5.10 (DS)
- net at IC5.9 (Q7): now also IC6.10 (DS)
- net DIR32: now reaches IC6.6 (D7)
- net DIR32: now also CON1.40
- net Shift_DATA: now reaches IC6.9 (Q7)
- new net DIR25: CON1.33, IC6.11 (D0)
- new net DIR26: CON1.34, IC6.12 (D1)
- new net DIR27: CON1.35, IC6.13 (D2)
- new net DIR28: CON1.36, IC6.14 (D3)
- new net DIR29: CON1.37, IC6.3 (D4)
- new net DIR30: CON1.38, IC6.4 (D5)
- new net DIR31: CON1.39, IC6.5 (D6)
- no-connect marks 0 -> 5
Other:
- moved on the sheet: IC5, IC6, IC7, IC8
