File: KiCAD Boards/LineFollower_V2/3_Current sense.kicad_sch (KiCad schematic)
At the start: 14 parts, among them IC10 LM358, IC11 INA199A3DCKR, IC12 INA199A3DCKR

Commit message: fix values, layout switchers
Parts:
- R21, R22: value 0Ω-1210 -> 0.02Ω-1210
- R23, R24: value 10K -> 1k

Commit message: ZubyMakove
Connections:
- net I_SENS_2_IN: no longer IC11.4 (IN+), R22.2
- net I_SENS_2_OUT: no longer IC11.5 (IN-), R22.1
- new net I_SENS_1_IN: IC11.4 (IN+), R22.2
- new net I_SENS_1_OUT: IC11.5 (IN-), R22.1

Commit message: v2 board 1.0
Connections:
- net I_SENS_2_IN: now also IC12.5 (IN-), R21.1; no longer IC12.4 (IN+), R21.2
- net I_SENS_2_OUT: now also IC12.4 (IN+), R21.2; no longer IC12.5 (IN-), R21.1
- net at IC10.5 (INPUT2(+): now also IC10.6 (INPUT2(-)), IC10.7 (OUTPUT2)
