File: KiCAD Boards/LineFollower_V2/4_Motor driver.kicad_sch (KiCad schematic)
At the start: 2 parts, among them CN1 HC-2510-2A, CN2 HC-2510-2A

Commit message: ZubyMakove
Parts:
- added C37, C38: 100n, Capacitor_SMD:C_0603_1608Metric, symbol Device:C
- added IC13, IC14: DRV8872DDAR, SOIC127P600X170-9N, symbol M4JCI:DRV8872DDAR
Connections:
- net I_SENS_1_OUT: now reaches CN1.1
- net IC_13_OUT_1: now reaches CN1.2
- net IC_13_OUT_1: now also IC13.6 (OUT1)
- net I_SENS_2_OUT: now reaches CN2.1
- net IC_14_OUT_2: now reaches CN2.2
- net IC_14_OUT_2: now also IC14.8 (OUT2)
- new net GND: C37.1, C38.1, IC13.1 (GND), IC13.7 (ISEN), IC13.9 (EP), IC14.1 (GND), IC14.7 (ISEN), IC14.9 (EP)
- new net I_SENS_1_IN: IC13.8 (OUT2)
- new net I_SENS_2_IN: IC14.6 (OUT1)
- new net L_IN_1: IC13.3 (IN1)
- new net L_IN_2: IC13.2 (IN2)
- new net R_IN_1: IC14.3 (IN1)
- new net R_IN_2: IC14.2 (IN2)
- new net VCC: C37.2, C38.2, IC13.5 (VM), IC14.5 (VM)
Other:
- moved on the sheet: CN2

Commit message: v2 board 1.0
Connections:
- net I_SENS_2_OUT: now also CN2.2; no longer CN2.1
- net IC_14_OUT_2 renamed IC_14_OUT
- net IC_14_OUT: now also CN2.1; no longer CN2.2
Changed lines of the file:
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@@
+	(wire
+		(pts
+			(xy 87.63 119.38) (xy 90.17 119.38)
+		)
+		(stroke
+			(width 0)
+			(type default)
+		)
+	)
 	(wire
 		(pts
@@
 	(wire
 		(pts
-			(xy 128.27 116.84) (xy 113.03 116.84)
-		)
-		(stroke
-			(width 0)
-			(type default)
-		)
-	)
-	(wire
-		(pts
-			(xy 113.03 116.84) (xy 113.03 114.3)
-		)
-		(stroke
-			(width 0)
-			(type default)
-		)
-	)
-	(wire
-		(pts
 			(xy 125.73 76.2) (xy 125.73 73.66)
 		)
@@
 	(wire
 		(pts
+			(xy 128.27 116.84) (xy 110.49 116.84)
+		)
+		(stroke
+			(width 0)
+			(type default)
+		)
+	)
+	(wire
+		(pts
 			(xy 72.39 93.98) (xy 72.39 96.52)
 		)
@@
 	(wire
 		(pts
+			(xy 110.49 114.3) (xy 87.63 114.3)
+		)
+		(stroke
+			(width 0)
+			(type default)
+		)
+	)
+	(wire
+		(pts
 			(xy 54.61 71.12) (xy 54.61 73.66)
 		)
@@
 	(wire
 		(pts
+			(xy 125.73 119.38) (xy 128.27 119.38)
+		)
+		(stroke
+			(width 0)
+			(type default)
+		)
+	)
+	(wire
+		(pts
 			(xy 123.19 73.66) (xy 125.73 73.66)
 		)
@@
 	(wire
 		(pts
-			(xy 113.03 114.3) (xy 87.63 114.3)
-		)
-		(stroke
-			(width 0)
-			(type default)
-		)
-	)
-	(wire
-		(pts
 			(xy 54.61 78.74) (xy 57.15 78.74)
 		)
@@
 	(wire
 		(pts
-			(xy 87.63 119.38) (xy 90.17 119.38)
+			(xy 110.49 116.84) (xy 110.49 114.3)
 		)
 		(stroke
@@
 		(pts
 			(xy 87.63 116.84) (xy 106.68 116.84)
-		)
-		(stroke
-			(width 0)
-			(type default)
-		)
-	)
-	(wire
-		(pts
-			(xy 125.73 119.38) (xy 128.27 119.38)
 		)
 		(stroke
@@
 		)
 	)
-	(label "IC_14_OUT_2"
-		(at 113.03 114.3 180)
+	(label "IC_14_OUT"
+		(at 110.49 114.3 0)
 		(fields_autoplaced yes)
 		(effects
@@
 				(size 1.27 1.27)
 			)
-			(justify right bottom)
+			(justify left bottom)
 		)
 	)
@@
 			)
 		)
-		(property "Description" "3.6A Brushed DC Motor Driver With Fault Reporting (PWM Ctrl) "
+		(property "Description" "3.6A Brushed DC Motor Driver With Fault Reporting (PWM Ctrl)"
 			(at 72.39 104.14 0)
 			(effects
@@
 		(lib_id "Robot druh-easyedapro:HC-2510-2A")
 		(at 133.35 118.11 0)
-		(mirror x)
 		(unit 1)
 		(exclude_from_sim no)
@@
 		(dnp no)
 		(property "Reference" "CN2"
-			(at 130.81 122.682 0)
+			(at 130.81 113.538 0)
 			(effects
 				(font
@@
 		)
 		(property "Value" "HC-2510-2A"
-			(at 130.81 111.76 0)
-			(effects
-				(font
+			(at 130.81 124.46 0)
+			(effects
+				(font
