File: KiCAD Boards/LineFollower_V2/LineFollower_V2.kicad_pcb (KiCad board)
At the start: 4 copper layers, 120 x 110 mm, 93 parts, among them CN1 HC-2510-2A, CN2 HC-2510-2A, CON1 XDFC-0520-40P, IC1 LF33CDT-TRY, IC10 LM358, IC11 INA199A3DCKR, IC12 INA199A3DCKR, IC2 2.4GHz, IC3 LMR36015FBRNXT, IC4 LMR36015FBRNXT, IC5 74HC165BQ,115, IC6 74HC165BQ,115, IC7 74HC165BQ,115, IC8 74HC165BQ,115, IC9 PCA9548APWR, Q1 BC817, Q2 BC817, SW1 TS3625A-HT, SW2 TS3625A-HT, U1 HC-VH-2A-TW, U2 DIP_2*5PIN_80MIL

Commit message: fix values, layout switchers
Parts:
- C1, C3: value 100nF -> 22uF; footprint Capacitor_SMD:C_0603_1608Metric -> Capacitor_SMD:C_0805_2012Metric; moved to B.Cu
- C10, C9: value 100nF -> 1uF
- C11, C14, C17, C19: value 100nF -> 220nF
- C12, C15, C18, C20, C23, C24, C25, C26: value 100nF -> 22uF; footprint Capacitor_SMD:C_0603_1608Metric -> Capacitor_SMD:C_0805_2012Metric
- C2, C4: value 100nF -> 220nF; moved to B.Cu
- C21, C22: value 100nF -> 20pF
- R1, R13, R14, R15, R16, R17, R18, R2: value 10K -> 5k1
- R10, R6, R7, R8: value 10K -> 100k
- R11: value 10K -> 24k9
- R21, R22: value 0Ω-1210 -> 0.02Ω-1210
- R23, R24: value 10K -> 1k
- R9: value 10K -> 43k2
- moved C7 186.3 mm to (166.0, 100.5), turned to -90 degrees
- moved SW1 182.6 mm to (162.5, 99.0), turned to -90 degrees
- moved C8 180.7 mm to (166.0, 87.5), turned to -90 degrees
- moved R3 179.4 mm to (166.0, 91.0), turned to -90 degrees
- moved SW2 178.5 mm to (162.5, 89.0), turned to 90 degrees
- moved C2 154.6 mm to (186.8, 79.5), turned to 180 degrees
- moved C1 154.6 mm to (187.0, 77.5), turned to 180 degrees
- moved C3 154.3 mm to (187.0, 81.5), turned to 180 degrees
- moved C4 154.1 mm to (187.0, 83.5), turned to 180 degrees
- moved R2 153.3 mm to (191.5, 82.3), turned to 90 degrees
- moved R1 153.1 mm to (191.5, 79.2), turned to -90 degrees
- moved IC2 153.0 mm to (177.1, 94.2), turned to -90 degrees
- moved USB1 141.8 mm to (197.4, 82.5), turned to 90 degrees
- moved L2 140.8 mm to (226.5, 57.8), turned to 90 degrees
- moved R7 137.0 mm to (227.5, 69.0), turned to 90 degrees
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Connections:
- C22 pad 1: <NO NET> -> +5V
- C24 pad 1: <NO NET> -> +5V
- C26 pad 1: <NO NET> -> +5V
- L2 pad 2: unconnected-(L2-Pad2) -> +5V
- LED10 pad 1: <NO NET> -> +5V
- LED11 pad 1: <NO NET> -> +5V
- LED12 pad 1: <NO NET> -> +5V
- LED3 pad 1: <NO NET> -> +5V
- LED4 pad 1: <NO NET> -> +5V
- LED5 pad 1: <NO NET> -> +5V
- LED6 pad 1: <NO NET> -> +5V
- LED7 pad 1: <NO NET> -> +5V
- LED8 pad 1: <NO NET> -> +5V
- LED9 pad 1: <NO NET> -> +5V
- R10 pad 2: <NO NET> -> +5V
Routing:
- net Net-(LED7-DIN): track 0.00 -> 55.8 mm

Commit message: some routing
Parts:
- added kibuzzard-669AC45D: G***, kibuzzard-669AC45D, F.Cu at (171.8, 100.8)
- added kibuzzard-669AC481: G***, kibuzzard-669AC481, F.Cu at (179.8, 100.8)
- C7, R1, R2: moved to B.Cu
- moved U2 230.7 mm to (126.5, 70.0)
- moved IC9 229.5 mm to (126.7, 78.9), turned to -90 degrees
- moved R12 225.4 mm to (120.8, 75.2), turned to 180 degrees
- moved R15 225.3 mm to (120.8, 81.2), turned to 180 degrees
- moved R16 225.0 mm to (120.8, 78.2), turned to 180 degrees
- moved R18 224.8 mm to (120.8, 79.7), turned to 180 degrees
- moved R17 224.8 mm to (120.8, 76.8), turned to 180 degrees
- moved C27 219.6 mm to (126.8, 74.0), turned to 180 degrees
- moved R14 213.1 mm to (132.8, 75.2), turned to 90 degrees
- moved R13 211.9 mm to (134.2, 76.2), turned to 90 degrees
- moved CN1 206.5 mm to (132.8, 130.8)
- moved LED2 202.9 mm to (170.1, 100.8), turned to 90 degrees
- moved C5 197.3 mm to (137.0, 60.8), turned to 90 degrees
- moved CN2 196.2 mm to (150.0, 130.7)
- moved C6 195.5 mm to (138.5, 60.8), turned to 90 degrees
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Connections:
- C21 pad 2: Net-(C21-Pad2) -> Net-(IC3-FB)
- C22 pad 2: Net-(C22-Pad2) -> Net-(IC4-FB)
- IC2 pad 28: unconnected-(IC2-IO35-Pad28) -> RGB_DATA
- IC5 pad 16: unconnected-(IC5-VCC-Pad16) -> 3V3
- IC6 pad 16: unconnected-(IC6-VCC-Pad16) -> 3V3
- IC7 pad 16: unconnected-(IC7-VCC-Pad16) -> 3V3
- IC8 pad 16: unconnected-(IC8-VCC-Pad16) -> 3V3
- L1 pad 2: unconnected-(L1-Pad2) -> 3V3_SWITCHING_OUT
- R10 pad 1: Net-(C22-Pad2) -> Net-(IC4-FB)
- R11 pad 1: Net-(IC4-FB) -> GND
- R11 pad 2: Net-(C22-Pad2) -> Net-(IC4-FB)
- R8 pad 1: Net-(C21-Pad2) -> Net-(IC3-FB)
- R9 pad 1: Net-(IC3-FB) -> GND
- R9 pad 2: Net-(C21-Pad2) -> Net-(IC3-FB)
Routing:
- net +5V: track 0.00 -> 97.7 mm, vias 0 -> 13
- net GND: track 0.00 -> 88.2 mm, vias 0 -> 72
- net VCC: track 0.00 -> 55.7 mm, vias 0 -> 18
- net RGB_DATA: track 0.00 -> 50.4 mm
- net USB_VBUS: track 0.00 -> 34.7 mm, vias 0 -> 3
- net 3V3_SWITCHING_OUT: track 0.00 -> 33.7 mm
- net 3V3_LDO_OUT: track 0.00 -> 20.2 mm
- net ESP_BOOT0: track 0.00 -> 19.1 mm, vias 0 -> 1
- net PG_5V: track 0.00 -> 16.4 mm, vias 0 -> 3
- net PG_3V3: track 0.00 -> 15.5 mm, vias 0 -> 2
- net Net-(IC3-VCC): track 0.00 -> 12.7 mm
- net ESP_RST: track 0.00 -> 11.2 mm
- net Net-(USB1-CC2): track 0.00 -> 8.27 mm, vias 0 -> 1
- net Net-(USB1-CC1): track 0.00 -> 7.58 mm, vias 0 -> 1
- net Net-(IC4-FB): track 0.00 -> 7.58 mm
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- added copper zone on B.Cu, net +5V
- added copper zone on B.Cu, net GND
- added copper zone on F.Cu, net GND
- added copper zone on B.Cu, net VCC
- added copper zone on F.Cu, net VCC

Commit message: more routing
Parts:
- added C33: 220nF, Capacitor_SMD:C_0603_1608Metric, F.Cu at (152.1, 40.3)
- added C34: 220nF, Capacitor_SMD:C_0603_1608Metric, F.Cu at (145.6, 45.8)
- added C35: 220nF, Capacitor_SMD:C_0603_1608Metric, F.Cu at (136.9, 46.5)
- added C36: 220nF, Capacitor_SMD:C_0603_1608Metric, F.Cu at (132.6, 40.0)
- added kibuzzard-669BBA84: G***, kibuzzard-669BBA84, F.Cu at (143.5, 84.8)
- C5, C6: value 100nF -> 1uF
- moved R1 115.4 mm to (84.4, 85.1), turned to 90 degrees
- moved R2 115.4 mm to (84.4, 82.1), turned to -90 degrees
- moved USB1 110.7 mm to (86.8, 83.7), turned to -90 degrees
- moved C4 87.6 mm to (98.7, 89.4), turned to 180 degrees
- moved C2 87.1 mm to (98.7, 85.3), turned to 180 degrees
- moved C3 86.9 mm to (98.9, 87.3), turned to 180 degrees
- moved C1 86.6 mm to (98.9, 83.3), turned to 180 degrees
- moved IC1 83.0 mm to (100.7, 85.9), turned to 180 degrees
- moved C24 37.3 mm to (192.1, 94.8), turned to 90 degrees
- moved R7 36.4 mm to (189.6, 82.2), turned to -90 degrees
- moved C20 35.7 mm to (191.4, 87.9), turned to 90 degrees
- moved C16 33.9 mm to (189.6, 85.2), turned to -90 degrees
- moved C10 32.4 mm to (188.1, 83.7), turned to 90 degrees
- moved C14 32.2 mm to (189.6, 88.2), turned to -90 degrees
- moved H1 31.6 mm to (143.5, 87.2), turned to 0 degrees
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Connections:
- CON1 pad 33: DIR17 -> DIR25
- CON1 pad 34: DIR18 -> DIR26
- CON1 pad 35: DIR19 -> DIR27
- CON1 pad 36: DIR20 -> DIR28
- CON1 pad 37: DIR21 -> DIR29
- CON1 pad 38: DIR22 -> DIR30
- CON1 pad 39: DIR23 -> DIR31
- CON1 pad 4: VCC -> 3V3
- CON1 pad 40: DIR24 -> DIR32
- CON1 pad 5: VCC -> 3V3
- IC2 pad 11: unconnected-(IC2-IO18-Pad11) -> I2C_RST
- IC2 pad 13: unconnected-(IC2-IO19-Pad13) -> USB_D+
- IC2 pad 14: unconnected-(IC2-IO20-Pad14) -> USB_D-
- IC2 pad 38: unconnected-(IC2-IO2-Pad38) -> CLK_Shift
- IC2 pad 39: unconnected-(IC2-IO1-Pad39) -> LOAD_Shift
- IC2 pad 4: unconnected-(IC2-IO4-Pad4) -> Shift_DATA
- IC2 pad 40: unconnected-(IC2-GND-Pad40) -> GND
- IC5 pad 1: unconnected-(IC5-PL#-Pad1) -> LOAD_Shift
- IC5 pad 10: unconnected-(IC5-DS-Pad10) -> Net-(IC5-DS)
- IC5 pad 15: unconnected-(IC5-CE#-Pad15) -> GND
- IC5 pad 17: unconnected-(IC5-PAD-Pad17) -> GND
- IC5 pad 2: unconnected-(IC5-CP-Pad2) -> CLK_Shift
- IC5 pad 9: unconnected-(IC5-Q7-Pad9) -> Net-(IC5-Q7)
- IC6 pad 1: unconnected-(IC6-PL#-Pad1) -> LOAD_Shift
- IC6 pad 10: unconnected-(IC6-DS-Pad10) -> Net-(IC5-Q7)
- IC6 pad 11: DIR17 -> DIR25
- IC6 pad 12: DIR18 -> DIR26
- IC6 pad 13: DIR19 -> DIR27
- IC6 pad 14: DIR20 -> DIR28
- IC6 pad 15: unconnected-(IC6-CE#-Pad15) -> GND
- IC6 pad 17: unconnected-(IC6-PAD-Pad17) -> GND
- IC6 pad 2: unconnected-(IC6-CP-Pad2) -> CLK_Shift
- IC6 pad 3: DIR21 -> DIR29
- IC6 pad 4: DIR22 -> DIR30
- IC6 pad 5: DIR23 -> DIR31
- IC6 pad 6: unconnected-(IC6-D7-Pad6) -> DIR32
- IC6 pad 9: unconnected-(IC6-Q7-Pad9) -> Shift_DATA
- IC7 pad 1: unconnected-(IC7-PL#-Pad1) -> LOAD_Shift
- IC7 pad 10: unconnected-(IC7-DS-Pad10) -> Net-(IC7-DS)
- IC7 pad 15: unconnected-(IC7-CE#-Pad15) -> GND
- IC7 pad 17: unconnected-(IC7-PAD-Pad17) -> GND
- IC7 pad 2: unconnected-(IC7-CP-Pad2) -> CLK_Shift
- IC7 pad 5: DIR14 -> DIR15
- IC7 pad 9: unconnected-(IC7-Q7-Pad9) -> Net-(IC5-DS)
- IC8 pad 1: unconnected-(IC8-PL#-Pad1) -> LOAD_Shift
- IC8 pad 15: unconnected-(IC8-CE#-Pad15) -> GND
- IC8 pad 17: unconnected-(IC8-PAD-Pad17) -> GND
- IC8 pad 2: unconnected-(IC8-CP-Pad2) -> CLK_Shift
- IC8 pad 9: unconnected-(IC8-Q7-Pad9) -> Net-(IC7-DS)
Routing:
- net GND: track 88.2 -> 401.2 mm, vias 72 -> 89
- net 3V3: track 5.62 -> 199.6 mm, vias 0 -> 10
- net CLK_Shift: track 0.00 -> 64.6 mm, vias 0 -> 5
- net LOAD_Shift: track 0.00 -> 63.9 mm, vias 0 -> 5
- net USB_D+: track 2.97 -> 62.1 mm, vias 1 -> 2
- net USB_D-: track 3.02 -> 55.8 mm, vias 1 -> 2
- net 3V3_LDO_OUT: track 20.2 -> 50.2 mm
- net Shift_DATA: track 0.00 -> 26.4 mm, vias 0 -> 2
- net VCC: track 55.7 -> 30.0 mm, vias 18 -> 19
- net +5V: track 97.7 -> 120.5 mm, vias 13 -> 17
- net I2C_RST: track 0.00 -> 22.7 mm
- net SCL: track 0.00 -> 17.7 mm
- net DIR24: track 0.00 -> 17.2 mm
- net DIR9: track 0.00 -> 16.6 mm
- net DIR23: track 0.00 -> 16.6 mm
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- added copper zone on F.Cu, net 3V3_SWITCHING_OUT

Commit message: ZubyMakove
Parts:
- added C37: 100n, Capacitor_SMD:C_0603_1608Metric, F.Cu at (102.5, 94.0)
- added C38: 100n, Capacitor_SMD:C_0603_1608Metric, F.Cu at (121.2, 92.2)
- added IC13: DRV8872DDAR, M4JCI:SOIC127P600X170-9N, F.Cu at (131.0, 94.6)
- added IC14: DRV8872DDAR, M4JCI:SOIC127P600X170-9N, F.Cu at (153.2, 93.5)
- moved R23 49.5 mm to (138.1, 98.2), turned to 90 degrees
- moved C31 48.8 mm to (140.8, 98.2), turned to 90 degrees
- moved C29 45.6 mm to (139.9, 100.9), turned to 0 degrees
- moved IC11 44.3 mm to (138.1, 103.0)
- moved R22 44.2 mm to (134.5, 102.6)
- moved CN2 28.5 mm to (154.2, 102.5), turned to 180 degrees
- moved CN1 28.3 mm to (129.9, 102.6), turned to 180 degrees
- moved C30 28.2 mm to (148.6, 112.2), turned to 180 degrees
- moved R21 26.1 mm to (144.2, 114.0)
- moved IC12 25.3 mm to (148.6, 114.3)
- moved C27 2.25 mm to (129.0, 74.0)
- moved R13 1.35 mm to (133.8, 77.5), turned to 0 degrees
- moved R12 1.25 mm to (120.0, 74.2)
- moved R14 1.25 mm to (133.8, 76.0), turned to 0 degrees
- moved R17 0.90 mm to (120.0, 76.2)
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Connections:
- CN1 pad 1: unconnected-(CN1-Pad1) -> I_SENS_1_OUT
- CN1 pad 2: unconnected-(CN1-Pad2) -> /Motor driver/IC_13_OUT_1
- CN2 pad 1: unconnected-(CN2-Pad1) -> I_SENS_2_OUT
- CN2 pad 2: unconnected-(CN2-Pad2) -> /Motor driver/IC_14_OUT_2
- IC11 pad 4: I_SENS_2_IN -> I_SENS_1_IN
- IC11 pad 5: I_SENS_2_OUT -> I_SENS_1_OUT
- R22 pad 1: I_SENS_2_OUT -> I_SENS_1_OUT
- R22 pad 2: I_SENS_2_IN -> I_SENS_1_IN
Routing:
- net GND: track 401.2 -> 300.0 mm, vias 89 -> 85
- net 3V3: track 199.6 -> 113.9 mm, vias 10 -> 8
- net SDA_R: track 2.96 -> 25.2 mm
- net I2C_RST: track 22.7 -> 4.80 mm
- net SDA_L: track 2.36 -> 16.7 mm
- net SCL_R: track 3.81 -> 14.3 mm
- net SCL_L: track 2.24 -> 11.3 mm
- net Net-(IC11-OUT): track 0.00 -> 5.32 mm
- net I_SENS_1_IN: track 0.00 -> 3.69 mm
- net I_SENS_1_OUT: track 0.00 -> 3.57 mm
- net I_SENS_1: track 0.00 -> 2.63 mm
- net SCL: track 17.7 -> 18.9 mm
- added copper zone on F.Cu, net /Motor driver/IC_13_OUT_1
- added copper zone on F.Cu, net I_SENS_1_IN
- added copper zone on F.Cu, net I_SENS_1_OUT

Commit message: v2 board 1.0
Parts:
- added CON1: XDFC-0520-40P, easyEDA_footprints:FPC-SMD_40P-P0.50_XDFC-0520-40P, F.Cu at (171.3, 23.4)
- added CON1: XDFC-0520-40P, easyEDA_footprints:AMPHENOL_62684-401100ALF, F.Cu at (171.3, 21.2)
- added G***: LOGO, M4JCI:Crow, F.Cu at (116.2, 122.8)
- added J1: Conn_01x10_Pin, Connector_PinHeader_2.54mm:PinHeader_1x10_P2.54mm_Vertical, F.Cu at (133.9, 83.0)
- added LED13: ~, easyEDA_footprints:LED0603-RD_GREEN, F.Cu at (130.7, 57.3)
- added LED14: ~, easyEDA_footprints:LED0603-RD_GREEN, F.Cu at (129.0, 57.3)
- added R25: 1K, Resistor_SMD:R_0603_1608Metric, F.Cu at (130.8, 60.3)
- added R26: 1K, Resistor_SMD:R_0603_1608Metric, F.Cu at (129.0, 60.4)
- added REF**: MountingHole_3.2mm_M3_Pad_Via, MountingHole:MountingHole_3.2mm_M3_Pad_Via, F.Cu at (178.8, 109.8)
- added REF**: MountingHole_3.2mm_M3_Pad_Via, MountingHole:MountingHole_3.2mm_M3_Pad_Via, F.Cu at (142.0, 126.1)
- added REF**: PinHeader_1x10_P2.54mm_Vertical, Connector_PinHeader_2.54mm:PinHeader_1x10_P2.54mm_Vertical, F.Cu at (121.0, 98.5)
- added REF**: PinHeader_1x10_P2.54mm_Vertical, Connector_PinHeader_2.54mm:PinHeader_1x10_P2.54mm_Vertical, F.Cu at (121.0, 96.0)
- added REF**: MountingHole_3.2mm_M3_Pad_Via, MountingHole:MountingHole_3.2mm_M3_Pad_Via, F.Cu at (160.2, 136.5)
- added REF**: MountingHole_3.2mm_M3_Pad_Via, MountingHole:MountingHole_3.2mm_M3_Pad_Via, F.Cu at (123.8, 136.5)
- added REF**: PinHeader_1x10_P2.54mm_Vertical, Connector_PinHeader_2.54mm:PinHeader_1x10_P2.54mm_Vertical, F.Cu at (121.0, 93.5)
- added REF**: MountingHole_3.2mm_M3_Pad_Via, MountingHole:MountingHole_3.2mm_M3_Pad_Via, F.Cu at (178.8, 136.6)
- added REF**: MountingHole_3.2mm_M3_Pad_Via, MountingHole:MountingHole_3.2mm_M3_Pad_Via, F.Cu at (105.2, 109.8)
- added REF**: PinHeader_1x10_P2.54mm_Vertical, Connector_PinHeader_2.54mm:PinHeader_1x10_P2.54mm_Vertical, F.Cu at (121.0, 103.6)
- added REF**: MountingHole_3.2mm_M3_Pad_Via, MountingHole:MountingHole_3.2mm_M3_Pad_Via, F.Cu at (105.2, 136.5)
- added REF**: MountingHole_3.2mm_M3_Pad_Via, MountingHole:MountingHole_3.2mm_M3_Pad_Via, F.Cu at (123.8, 109.8)
- added REF**: PinHeader_1x10_P2.54mm_Vertical, Connector_PinHeader_2.54mm:PinHeader_1x10_P2.54mm_Vertical, F.Cu at (121.0, 101.1)
- added REF**: MountingHole_3.2mm_M3_Pad_Via, MountingHole:MountingHole_3.2mm_M3_Pad_Via, F.Cu at (142.0, 136.0)
- added REF**: MountingHole_3.2mm_M3_Pad_Via, MountingHole:MountingHole_3.2mm_M3_Pad_Via, F.Cu at (160.2, 109.8)
- added kibuzzard-669E1D82: G***, kibuzzard-669E1D82, F.Cu at (126.2, 100.8)
- added kibuzzard-669E1D82: G***, kibuzzard-669E1D82, F.Cu at (157.8, 100.5)
- added kibuzzard-669E1EE7: G***, kibuzzard-669E1EE7, F.Cu at (136.5, 80.8)
- added kibuzzard-669E1EEE: G***, kibuzzard-669E1EEE, F.Cu at (139.0, 80.8)
- added kibuzzard-669E1EFC: G***, kibuzzard-669E1EFC, F.Cu at (141.6, 80.8)
- added kibuzzard-669E1F08: G***, kibuzzard-669E1F08, F.Cu at (144.1, 80.8)
- added kibuzzard-669E1F0E: G***, kibuzzard-669E1F0E, F.Cu at (146.6, 80.8)
- added kibuzzard-669E1F1F: G***, kibuzzard-669E1F1F, F.Cu at (149.2, 80.8)
- added kibuzzard-669E1F24: G***, kibuzzard-669E1F24, F.Cu at (151.7, 80.8)
- added kibuzzard-669E1F2D: G***, kibuzzard-669E1F2D, F.Cu at (154.2, 80.8)
- added kibuzzard-669E1F34: G***, kibuzzard-669E1F34, F.Cu at (156.8, 80.8)
- added kibuzzard-669E1F50: G***, kibuzzard-669E1F50, F.Cu at (134.0, 80.8)
- added kibuzzard-669E1FB3: G***, kibuzzard-669E1FB3, F.Cu at (127.5, 63.5)
- added kibuzzard-669E206F: G***, kibuzzard-669E206F, F.Cu at (164.5, 71.8)
- added kibuzzard-669E2084: G***, kibuzzard-669E2084, F.Cu at (127.2, 66.2)
- added kibuzzard-669E2110: G***, kibuzzard-669E2110, F.Cu at (196.2, 87.8)
- added kibuzzard-669E2194: G***, kibuzzard-669E2194, F.Cu at (201.0, 81.8)
- added kibuzzard-669E23C8: G***, kibuzzard-669E23C8, F.Cu at (129.0, 52.5)
- added kibuzzard-669E23CE: G***, kibuzzard-669E23CE, F.Cu at (130.8, 53.1)
- C1, C2, C3, C4, C7: moved to F.Cu
- moved C37 46.9 mm to (149.4, 92.8), turned to -90 degrees
- moved C32 40.5 mm to (146.0, 96.5), turned to 180 degrees
- moved R24 38.1 mm to (146.0, 98.1), turned to 180 degrees
- moved kibuzzard-669AC481 34.4 mm to (195.2, 101.8)
- moved LED1 31.2 mm to (193.2, 103.3)
- moved R4 31.2 mm to (193.2, 100.4)
- moved R20 30.0 mm to (139.3, 114.5), turned to 0 degrees
- moved C28 26.6 mm to (139.8, 107.0), turned to 180 degrees
- moved IC10 25.9 mm to (142.5, 110.8), turned to -90 degrees
- moved kibuzzard-669AC45D 25.3 mm to (191.2, 101.8), turned to 90 degrees
- moved R19 25.1 mm to (142.5, 114.5), turned to 0 degrees
- moved LED2 24.7 mm to (189.3, 103.4), turned to 90 degrees
- moved R5 19.7 mm to (189.3, 100.4), turned to 90 degrees
- moved R21 14.2 mm to (149.6, 100.9), turned to -90 degrees
- moved IC12 14.0 mm to (146.0, 100.5), turned to 180 degrees
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Connections:
- CN2 pad 1: I_SENS_2_OUT -> /Motor driver/IC_14_OUT
- CN2 pad 2: /Motor driver/IC_14_OUT_2 -> I_SENS_2_OUT
- IC10 pad 5: unconnected-(IC10B-INPUT2(+-Pad5) -> Net-(IC10B-INPUT2(+)
- IC10 pad 6: unconnected-(IC10B-INPUT2(-)-Pad6) -> Net-(IC10B-INPUT2(+)
- IC10 pad 7: unconnected-(IC10B-OUTPUT2-Pad7) -> Net-(IC10B-INPUT2(+)
- IC12 pad 4: I_SENS_2_IN -> I_SENS_2_OUT
- IC12 pad 5: I_SENS_2_OUT -> I_SENS_2_IN
- IC14 pad 8: /Motor driver/IC_14_OUT_2 -> /Motor driver/IC_14_OUT
- IC2 pad 18: unconnected-(IC2-IO10-Pad18) -> L_IN_1
- IC2 pad 19: unconnected-(IC2-IO11-Pad19) -> L_IN_2
- IC2 pad 20: unconnected-(IC2-IO12-Pad20) -> IO12
- IC2 pad 21: unconnected-(IC2-IO13-Pad21) -> I_SENS_1
- IC2 pad 22: unconnected-(IC2-IO14-Pad22) -> I_SENS_2
- IC2 pad 23: unconnected-(IC2-IO21-Pad23) -> R_IN_1
- IC2 pad 24: unconnected-(IC2-IO33-Pad24) -> R_IN_2
- IC2 pad 25: unconnected-(IC2-IO34-Pad25) -> IO34
- IC2 pad 29: unconnected-(IC2-IO36-Pad29) -> IO36
- IC2 pad 30: unconnected-(IC2-IO37-Pad30) -> IO37
- IC2 pad 5: unconnected-(IC2-IO5-Pad5) -> Led_Sig_1
- IC2 pad 6: unconnected-(IC2-IO6-Pad6) -> Led_Sig_2
- R21 pad 1: I_SENS_2_OUT -> I_SENS_2_IN
- R21 pad 2: I_SENS_2_IN -> I_SENS_2_OUT
Routing:
- net 3V3: track 113.9 -> 247.9 mm, vias 8 -> 12
- net GND: track 300.0 -> 182.5 mm, vias 85 -> 240
- net Net-(LED2-C): track 2.17 -> 34.8 mm, vias 0 -> 2
- net Net-(LED1-C): track 2.13 -> 33.7 mm
- net USB_VBUS: track 33.8 -> 3.20 mm, vias 3 -> 0
- net I_SENS_1: track 2.63 -> 28.0 mm
- net I_SENS_2: track 0.00 -> 24.3 mm
- net L_IN_2: track 0.00 -> 24.2 mm
- net L_IN_1: track 0.00 -> 24.2 mm
- net VCC: track 30.0 -> 52.6 mm, vias 19 -> 26
- net I2C_RST: track 4.80 -> 26.9 mm, vias 0 -> 2
- net MIDPOINT_REF: track 0.00 -> 15.4 mm, vias 0 -> 2
- net R_IN_1: track 0.00 -> 14.7 mm
- net Led_Sig_2: track 0.00 -> 14.1 mm
- net R_IN_2: track 0.00 -> 13.7 mm
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- added copper zone on F.Cu, net /Motor driver/IC_14_OUT
- added copper zone on F.Cu, net I_SENS_2_IN
- added copper zone on F.Cu, net I_SENS_2_OUT
- added copper zone on F.Cu, net USB_VBUS
Other:
- outline, holes or cut-outs redrawn
- copper layers 4 -> 2
- board text added: "JLCJLCJLCJLC"
- board text added: "Skibidi"
- board text added: "WayWayWay"
